File: beeper/beeper.brd (EAGLE design)
At the start: 45.4 x 80 mm, 13 parts, among them IC1 LM555N, IC2 LM555N, U1 CD4011BE

Commit message: completed CAM
Parts:
- removed IC1, IC2: LM555N, linear:DIL08
- removed LS1: AI-2331-TWT-R, AI-2331-TWT-R:XDCR_AI-2331-TWT-R
- added BZ: F/QMBIII, buzzer:F/QMBIII
- added GND, VCC: (no value), wirepad:SMD1,27-2,54
- added U2, U3: LMC555CN, LMC555CN:DIP794W45P254L959H508Q8
- moved R4 6.35 mm to (10.2, 55.9)
- moved R3 4.58 mm to (39.4, 55.9)
- moved C1 1.27 mm to (38.1, 17.8)
Connections:
- net GND: now also GND.1, U2.1, U3.1; no longer IC1.1, IC2.1
- net N$1: now also U2.7; no longer IC1.7
- net N$10: now also BZ.-; no longer LS1.P
- net N$2: now also U2.2, U2.6; no longer IC1.2, IC1.6
- net N$3: now also U2.3; no longer IC1.3
- net N$5: now also R3.1, R6.3, U3.7; no longer C2.1, IC2.2, IC2.6, R6.1, R6.2
- net N$6: now also C2.1, R6.1, R6.2, U3.2, U3.6; no longer IC2.7, R3.1, R6.3
- net N$8: now also U3.3; no longer IC2.3
- net VCC: now also BZ.+, U2.4, U2.8, U3.4, U3.8, VCC.1; no longer IC1.4, IC1.8, IC2.4, IC2.8, LS1.N
Routing:
- net N$6: track 55.0 -> 76.6 mm
- net N$3: track 87.9 -> 73.5 mm
- net VCC: track 109.7 -> 106.7 mm, vias 1 -> 0
- net N$5: track 61.2 -> 60.7 mm
