File: beeper/beeper.sch (EAGLE design)
At the start: 13 parts, among them IC1 LM555N, IC2 LM555N, U1 CD4011BE

Commit message: completed CAM
Parts:
- removed IC1, IC2: LM555N, linear:LM555N
- removed LS1: AI-2331-TWT-R, AI-2331-TWT-R:AI-2331-TWT-R
- added BZ: F/QMBIII, buzzer:F/QMBIII
- added GND, VCC: (no value), wirepad:SMD2
- added U2, U3: LMC555CN, LMC555CN:LMC555CN
Connections:
- net GND: now also GND.P, U2.GND, U3.GND; no longer IC1.GND, IC2.GND
- net N$1: now also U2.DISCHARGE; no longer IC1.DIS
- net N$10: now also BZ.+; no longer LS1.+
- net N$2: now also U2.THRESHOLD, U2.TRIGGER; no longer IC1.THR, IC1.TR
- net N$3: now also U2.OUTPUT; no longer IC1.Q
- net N$5: now also R3.1, R6.3, U3.DISCHARGE; no longer C2.1, IC2.THR, IC2.TR, R6.1, R6.2
- net N$6: now also C2.1, R6.1, R6.2, U3.THRESHOLD, U3.TRIGGER; no longer IC2.DIS, R3.1, R6.3
- net N$8: now also U3.OUTPUT; no longer IC2.Q
- net VCC: now also BZ.-, U2.RESET, U2.V+, U3.RESET, U3.V+, VCC.P; no longer IC1.R, IC1.V+, IC2.R, IC2.V+, LS1.-
Other:
- moved on the sheet: C1, C2, LED1, R1, R2, R3, R5, R6
